File: ads7886_PCB/ads7886.kicad_pcb (KiCad board)
At the start: 2 copper layers, 38.5 x 13.5 mm, 23 parts, among them IC1 ADS7886SDBVT, J1 2214S-08SG-85, J2 2214S-08SG-85, U1 LP5907MFX-3.3, U2 OPA355NA, U3 74LVC1G14

Commit message: Improved PCB component compatilibity
Widened LDO trace between IN and EN, mostly for aesthetics
Grounded previously NC pad on inverter to allow for optional installation of 1G240 instead of 1G14
Parts:
- U3: value 74LVC1G14 -> 74LVC1G240
Connections:
- J1 pad 6: (no net) -> Net-(J1-Pad6)
- J2 pad 1: (no net) -> Net-(J2-Pad1)
- J2 pad 4: (no net) -> Net-(J2-Pad4)
- R2 pad 3: (no net) -> Net-(R2-Pad3)
- U1 pad 4: (no net) -> Net-(U1-Pad4)
- U3 pad 1: (no net) -> GND
Other:
- board text added: "ADC Mezzanine 0.5"
- board text removed: "ADC Mezzanine 0.4"
Changed lines of the file:
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@@
     (zones 0)
     (modules 23)
-    (nets 14)
+    (nets 19)
   )
   (page A4)
@@
   (net 12 /PD)
   (net 13 "Net-(R3-Pad2)")
+  (net 14 "Net-(J1-Pad6)")
+  (net 15 "Net-(J2-Pad1)")
+  (net 16 "Net-(J2-Pad4)")
+  (net 17 "Net-(R2-Pad3)")
+  (net 18 "Net-(U1-Pad4)")
   (net_class Default "This is the default net class."
     (clearance 0.2)
@@
     (add_net GND)
     (add_net "Net-(D1-Pad2)")
+    (add_net "Net-(J1-Pad6)")
+    (add_net "Net-(J2-Pad1)")
+    (add_net "Net-(J2-Pad4)")
+    (add_net "Net-(R2-Pad3)")
     (add_net "Net-(R3-Pad2)")
+    (add_net "Net-(U1-Pad4)")
     (add_net VCC)
   )
@@
     (fp_line (start 9.19 -3.81) (end -1.27 -3.81) (layer F.SilkS) (width 0.2))
     (fp_line (start -1.27 -3.81) (end -1.27 0) (layer F.SilkS) (width 0.2))
-    (pad 1 thru_hole rect (at 0 0 90) (size 1.575 1.575) (drill 1.05) (layers *.Cu *.Mask F.SilkS))
+    (pad 1 thru_hole rect (at 0 0 90) (size 1.575 1.575) (drill 1.05) (layers *.Cu *.Mask F.SilkS)
+      (net 15 "Net-(J2-Pad1)"))
     (pad 2 thru_hole circle (at 0 -2.54 90) (size 1.575 1.575) (drill 1.05) (layers *.Cu *.Mask F.SilkS)
       (net 10 GND))
     (pad 3 thru_hole circle (at 2.54 0 90) (size 1.575 1.575) (drill 1.05) (layers *.Cu *.Mask F.SilkS)
       (net 6 /SDO))
-    (pad 4 thru_hole circle (at 2.54 -2.54 90) (size 1.575 1.575) (drill 1.05) (layers *.Cu *.Mask F.SilkS))
+    (pad 4 thru_hole circle (at 2.54 -2.54 90) (size 1.575 1.575) (drill 1.05) (layers *.Cu *.Mask F.SilkS)
+      (net 16 "Net-(J2-Pad4)"))
     (pad 5 thru_hole circle (at 5.08 0 90) (size 1.575 1.575) (drill 1.05) (layers *.Cu *.Mask F.SilkS)
       (net 8 /LATCH))
@@
     (pad 7 thru_hole circle (at 7.62 0 180) (size 1.575 1.575) (drill 1.05) (layers *.Cu *.Mask F.SilkS)
       (net 2 /5VA))
-    (pad 6 thru_hole circle (at 5.08 -2.54 180) (size 1.575 1.575) (drill 1.05) (layers *.Cu *.Mask F.SilkS))
+    (pad 6 thru_hole circle (at 5.08 -2.54 180) (size 1.575 1.575) (drill 1.05) (layers *.Cu *.Mask F.SilkS)
+      (net 14 "Net-(J1-Pad6)"))
     (pad 5 thru_hole circle (at 5.08 0 180) (size 1.575 1.575) (drill 1.05) (layers *.Cu *.Mask F.SilkS)
       (net 9 /SIG_IN))
@@
     (pad 2 smd rect (at 0 -1.55 90) (size 1.5 1.6) (layers F.Cu F.Paste F.Mask)
       (net 4 /VIN))
-    (pad 3 smd rect (at 1 1.7 90) (size 1.2 1.2) (layers F.Cu F.Paste F.Mask))
+    (pad 3 smd rect (at 1 1.7 90) (size 1.2 1.2) (layers F.Cu F.Paste F.Mask)
+      (net 17 "Net-(R2-Pad3)"))
     (model C:/SamacSys_PCB_Library/KiCad/SamacSys_Parts.3dshapes/TC33X-2-101E.stp
       (at (xyz 0 0 0))
@@
     (pad 3 smd rect (at -1.35 -0.95) (size 1.56 0.65) (layers B.Cu B.Paste B.Mask)
       (net 2 /5VA))
-    (pad 4 smd rect (at 1.35 -0.95) (size 1.56 0.65) (layers B.Cu B.Paste B.Mask))
+    (pad 4 smd rect (at 1.35 -0.95) (size 1.56 0.65) (layers B.Cu B.Paste B.Mask)
+      (net 18 "Net-(U1-Pad4)"))
     (pad 5 smd rect (at 1.35 0.95) (size 1.56 0.65) (layers B.Cu B.Paste B.Mask)
       (net 1 /VDD))
-    (model ${KISYS3DMOD}/TO_SOT_Packages_SMD.3dshapes\SOT-23-5.wrl
-      (at (xyz 0 0 0))
-      (scale (xyz 1 1 1))
-      (rotate (xyz 0 0 0))
-    )
-  )
-  (module TO_SOT_Packages_SMD:SOT-23-5_HandSoldering (layer B.Cu)
-    (at 161.036 94.234)
-    (descr "5-pin SOT23 package")
-    (tags "SOT-23-5 hand-soldering")
-    (attr smd)
-    (fp_text reference U3 (at -3.429 -1.016 -180) (layer B.SilkS)
-      (effects (font (size 1 1) (thickness 0.15)) (justify mirror))
-    )
-    (fp_text value 74LVC1G14 (at 0 -2.9 -180) (layer B.Fab)
-      (effects (font (size 1 1) (thickness 0.15)) (justify mirror))
-    )
-    (fp_line (start 2.38 -1.8) (end -2.38 -1.8) (layer B.CrtYd) (width 0.05))
-    (fp_line (start 2.38 -1.8) (end 2.38 1.8) (layer B.CrtYd) (width 0.05))
-    (fp_line (start -2.38 1.8) (end -2.38 -1.8) (layer B.CrtYd) (width 0.05))
-    (fp_line (start -2.38 1.8) (end 2.38 1.8) (layer B.CrtYd) (width 0.05))
-    (fp_line (start 0.9 1.55) (end 0.9 -1.55) (layer B.Fab) (width 0.1))
-    (fp_line (start 0.9 -1.55) (end -0.9 -1.55) (layer B.Fab) (width 0.1))
-    (fp_line (start -0.9 0.9) (end -0.9 -1.55) (layer B.Fab) (width 0.1))
-    (fp_line (start 0.9 1.55) (end -0.25 1.55) (layer B.Fab) (width 0.1))
-    (fp_line (start -0.9 0.9) (end -0.25 1.55) (layer B.Fab) (width 0.1))
-    (fp_line (start 0.9 1.61) (end -1.55 1.61) (layer B.SilkS) (width 0.12))
-    (fp_line (start -0.9 -1.61) (end 0.9 -1.61) (layer B.SilkS) (width 0.12))
-    (fp_text user %R (at 0 0 -270) (layer B.Fab)
-      (effects (font (size 0.5 0.5) (thickness 0.075)) (justify mirror))
-    )
-    (pad 5 smd rect (at 1.35 0.95) (size 1.56 0.65) (layers B.Cu B.Paste B.Mask)
-      (net 11 VCC))
-    (pad 4 smd rect (at 1.35 -0.95) (size 1.56 0.65) (layers B.Cu B.Paste B.Mask)
-      (net 13 "Net-(R3-Pad2)"))
-    (pad 3 smd rect (at -1.35 -0.95) (size 1.56 0.65) (layers B.Cu B.Paste B.Mask)
-      (net 10 GND))
-    (pad 2 smd rect (at -1.35 0) (size 1.56 0.65) (layers B.Cu B.Paste B.Mask)
-      (net 8 /LATCH))
-    (pad 1 smd rect (at -1.35 0.95) (size 1.56 0.65) (layers B.Cu B.Paste B.Mask))
     (model ${KISYS3DMOD}/TO_SOT_Packages_SMD.3dshapes\SOT-23-5.wrl
       (at (xyz 0 0 0))
@@
     )
   )
-  (gr_text "ADC Mezzanine 0.4" (at 135.128 102.362) (layer F.SilkS)
+  (module TO_SOT_Packages_SMD:SOT-23-5_HandSoldering (layer B.Cu)
+    (at 161.036 94.234)
+    (descr "5-pin SOT23 package")
+    (tags "SOT-23-5 hand-soldering")
+    (attr smd)
+    (fp_text reference U3 (at 0 2.9) (layer B.SilkS)
+      (effects (font (size 1 1) (thickness 0.15)) (justify mirror))
+    )
+    (fp_text value 74LVC1G240 (at 0 -2.9) (layer B.Fab)
+      (effects (font (size 1 1) (thickness 0.15)) (justify mirror))
+    )
+    (fp_line (start 2.38 -1.8) (end -2.38 -1.8) (layer B.CrtYd) (width 0.05))
+    (fp_line (start 2.38 -1.8) (end 2.38 1.8) (layer B.CrtYd) (width 0.05))
+    (fp_line (start -2.38 1.8) (end -2.38 -1.8) (layer B.CrtYd) (width 0.05))
+    (fp_line (start -2.38 1.8) (end 2.38 1.8) (layer B.CrtYd) (width 0.05))
+    (fp_line (start 0.9 1.55) (end 0.9 -1.55) (layer B.Fab) (width 0.1))
+    (fp_line (start 0.9 -1.55) (end -0.9 -1.55) (layer B.Fab) (width 0.1))
+    (fp_line (start -0.9 0.9) (end -0.9 -1.55) (layer B.Fab) (width 0.1))
+    (fp_line (start 0.9 1.55) (end -0.25 1.55) (layer B.Fab) (width 0.1))
+    (fp_line (start -0.9 0.9) (end -0.25 1.55) (layer B.Fab) (width 0.1))
+    (fp_line (start 0.9 1.61) (end -1.55 1.61) (layer B.SilkS) (width 0.12))
+    (fp_line (start -0.9 -1.61) (end 0.9 -1.61) (layer B.SilkS) (width 0.12))
+    (fp_text user %R (at 0 0 -90) (layer B.Fab)
+      (effects (font (size 0.5 0.5) (thickness 0.075)) (justify mirror))
+    )
+    (pad 5 smd rect (at 1.35 0.95) (size 1.56 0.65) (layers B.Cu B.Paste B.Mask)
+      (net 11 VCC))
+    (pad 4 smd rect (at 1.35 -0.95) (size 1.56 0.65) (layers B.Cu B.Paste B.Mask)
+      (net 13 "Net-(R3-Pad2)"))
+    (pad 3 smd rect (at -1.35 -0.95) (size 1.56 0.65) (layers B.Cu B.Paste B.Mask)
+      (net 10 GND))
+    (pad 2 smd rect (at -1.35 0) (size 1.56 0.65) (layers B.Cu B.Paste B.Mask)
+      (net 8 /LATCH))
+    (pad 1 smd rect (at -1.35 0.95) (size 1.56 0.65) (layers B.Cu B.Paste B.Mask)
+      (net 10 GND))
+    (model ${KISYS3DMOD}/TO_SOT_Packages_SMD.3dshapes\SOT-23-5.wrl
+      (at (xyz 0 0 0))
+      (scale (xyz 1 1 1))
+      (rotate (xyz 0 0 0))
+    )
+  )
+  (gr_text "ADC Mezzanine 0.5" (at 135.128 102.362) (layer F.SilkS)
     (effects (font (size 1 1) (thickness 0.15)))
   )
@@
   (segment (start 133.985 92.395) (end 135.048 92.395) (width 0.508) (layer B.Cu) (net 2))
   (segment (start 131.445 91.694) (end 128.905 91.694) (width 0.508) (layer F.Cu) (net 2))
-  (segment (start 136.9964 95.311) (end 136.064 95.311) (width 0.1524) (layer B.Cu) (net 2))
-  (segment (start 137.120201 95.187199) (end 136.9964 95.311) (width 0.1524) (layer B.Cu) (net 2))
-  (segment (start 137.120201 93.534801) (end 137.120201 95.187199) (width 0.1524) (layer B.Cu) (net 2))
-  (segment (start 136.9964 93.411) (end 137.120201 93.534801) (width 0.1524) (layer B.Cu) (net 2))
-  (segment (start 136.064 93.411) (end 136.9964 93.411) (width 0.1524) (layer B.Cu) (net 2))
+  (segment (start 137.098 95.311) (end 136.064 95.311) (width 0.254) (layer B.Cu) (net 2))
+  (segment (start 137.171001 95.237999) (end 137.098 95.311) (width 0.254) (layer B.Cu) (net 2))
+  (segment (start 137.171001 93.774399) (end 137.171001 95.237999) (width 0.254) (layer B.Cu) (net 2))
+  (segment (start 136.807602 93.411) (end 137.171001 93.774399) (width 0.254) (layer B.Cu) (net 2))
+  (segment (start 136.064 93.411) (end 136.807602 93.411) (width 0.254) (layer B.Cu) (net 2))
   (via (at 134.62 101.473) (size 0.762) (drill 0.508) (layers F.Cu B.Cu) (net 3))
   (segment (start 135.636 100.922) (end 135.171 100.922) (width 0.508) (layer F.Cu) (net 3))
